File: MIDI.sch (KiCad schematic (older format))
At the start: 9 parts, among them J13 57PC5F, J14 57PC5F, U2 6N138SDM

Commit message: Updated MIDI schematic and orientation and to do list. Note: Gerber not updated.
Parts:
- removed R10, R11: 47, SamacSys_Parts:R_0805_JLCPCB, symbol JLCPBC_Basic:47
- added R10: 33, SamacSys_Parts:R_0805_JLCPCB, symbol JLCPBC_Basic:33
- added R11: 10, SamacSys_Parts:R_1206_JLCPCB, symbol JLCPBC_Basic:10
Connections:
- net labels removed: +5V
Changed lines of the file:
@@
 NoConn ~ 1600 2600
 NoConn ~ 1600 2700
-Text HLabel 8950 2700 2    50   Input ~ 0
+Text HLabel 8950 3050 2    50   Input ~ 0
 MIDI_OUT
 $Comp
@@
 	1    0    0    -1
 $EndComp
-$Comp
-L power:+5V #PWR044
-U 1 1 5F6AFFEE
-P 8950 3050
-F 0 "#PWR044" H 8950 2900 50  0001 C CNN
-F 1 "+5V" H 8965 3223 50  0000 C CNN
-F 2 "" H 8950 3050 50  0001 C CNN
-F 3 "" H 8950 3050 50  0001 C CNN
-	1    8950 3050
-	1    0    0    -1
-$EndComp
-$Comp
-L JLCPBC_Basic:47 R10
-U 1 1 5F6B545F
-P 8350 2700
-F 0 "R10" H 8500 2800 50  0000 C CNN
-F 1 "47" H 8500 2600 50  0000 C CNN
-F 2 "SamacSys_Parts:R_0805_JLCPCB" H 8900 2750 50  0001 L CNN
-F 3 "https://datasheet.lcsc.com/szlcsc/Uniroyal-Elec-0805W8F470JT5E_C17714.pdf" H 8900 2650 50  0001 L CNN
-F 4 "Chip Resistor - Surface Mount 47Ohms ±1% 1/8W 0805 RoHS" H 8900 2550 50  0001 L CNN "Description"
-F 5 "UNI-ROYAL(Uniroyal Elec)" H 8900 2150 50  0001 L CNN "Manufacturer_Name"
-F 6 "0805W8F470JT5E" H 8900 2050 50  0001 L CNN "Manufacturer_Part_Number"
-F 7 "C17714" H 8350 2700 50  0001 C CNN "JLCPCB Part Number"
-	1    8350 2700
-	1    0    0    -1
-$EndComp
-$Comp
-L JLCPBC_Basic:47 R11
-U 1 1 5F6B6CD0
-P 8350 3050
-F 0 "R11" H 8500 3150 50  0000 C CNN
-F 1 "47" H 8500 2950 50  0000 C CNN
-F 2 "SamacSys_Parts:R_0805_JLCPCB" H 8900 3100 50  0001 L CNN
-F 3 "https://datasheet.lcsc.com/szlcsc/Uniroyal-Elec-0805W8F470JT5E_C17714.pdf" H 8900 3000 50  0001 L CNN
-F 4 "Chip Resistor - Surface Mount 47Ohms ±1% 1/8W 0805 RoHS" H 8900 2900 50  0001 L CNN "Description"
-F 5 "UNI-ROYAL(Uniroyal Elec)" H 8900 2500 50  0001 L CNN "Manufacturer_Name"
-F 6 "0805W8F470JT5E" H 8900 2400 50  0001 L CNN "Manufacturer_Part_Number"
-F 7 "C17714" H 8350 3050 50  0001 C CNN "JLCPCB Part Number"
-	1    8350 3050
-	1    0    0    -1
-$EndComp
 Wire Wire Line
 	7900 2700 8350 2700
@@
 	4950 2150 4950 2100
 Connection ~ 4950 2150
+$Comp
+L power:+3.3V #PWR?
+U 1 1 5FE8AA11
+P 8950 2700
+AR Path="/5FE8AA11" Ref="#PWR?"  Part="1"
+AR Path="/5F699A2B/5FE8AA11" Ref="#PWR0101"  Part="1"
+F 0 "#PWR0101" H 8950 2550 50  0001 C CNN
+F 1 "+3.3V" H 8965 2873 50  0000 C CNN
+F 2 "" H 8950 2700 50  0001 C CNN
+F 3 "" H 8950 2700 50  0001 C CNN
+	1    8950 2700
+	1    0    0    -1
+$EndComp
+$Comp
+L JLCPBC_Basic:33 R10
+U 1 1 5FE8D1EA
+P 8350 2700
+F 0 "R10" H 8500 2907 50  0000 C CNN
+F 1 "33" H 8500 2816 50  0000 C CNN
+F 2 "SamacSys_Parts:R_0805_JLCPCB" H 8900 2750 50  0001 L CNN
+F 3 "https://datasheet.lcsc.com/szlcsc/Uniroyal-Elec-0805W8F330JT5E_C17634.pdf" H 8900 2650 50  0001 L CNN
+F 4 "Chip Resistor - Surface Mount 33Ohms ±1% 1/8W 0805 RoHS" H 8900 2550 50  0001 L CNN "Description"
+F 5 "UNI-ROYAL(Uniroyal Elec)" H 8900 2150 50  0001 L CNN "Manufacturer_Name"
+F 6 "0805W8F330JT5E" H 8900 2050 50  0001 L CNN "Manufacturer_Part_Number"
+F 7 "C17634" H 8350 2700 50  0001 C CNN "JLCPCB Part Number"
+	1    8350 2700
+	1    0    0    -1
+$EndComp
+$Comp
+L JLCPBC_Basic:10 R11
+U 1 1 5FE8D9B0
+P 8350 3050
+F 0 "R11" H 8500 3257 50  0000 C CNN
+F 1 "10" H 8500 3166 50  0000 C CNN
+F 2 "SamacSys_Parts:R_1206_JLCPCB" H 8900 3100 50  0001 L CNN
+F 3 "https://datasheet.lcsc.com/szlcsc/Uniroyal-Elec-1206W4F100JT5E_C17903.pdf" H 8900 3000 50  0001 L CNN
+F 4 "Chip Resistor - Surface Mount 10Ohms ±1% 1/4W 1206 RoHS" H 8900 2900 50  0001 L CNN "Description"
+F 5 "UNI-ROYAL(Uniroyal Elec)" H 8900 2500 50  0001 L CNN "Manufacturer_Name"
+F 6 "1206W4F100JT5E" H 8900 2400 50  0001 L CNN "Manufacturer_Part_Number"
+F 7 "C17903" H 8350 3050 50  0001 C CNN "JLCPCB Part Number"
+	1    8350 3050
+	1    0    0    -1
+$EndComp
 $EndSCHEMATC

Commit message: Replaced one pot by a 3.5mm MIDI Output jack.
Parts:
- added J?: SJ1-3523N, SJ13523N, symbol SamacSys_Parts:SJ1-3523N
- added R?: 10, SamacSys_Parts:R_1206_JLCPCB, symbol JLCPBC_Basic:10
- added R?: 33, SamacSys_Parts:R_0805_JLCPCB, symbol JLCPBC_Basic:33
Connections:
- net labels added: MIDI_OUT2
- wire segments 36 -> 41
- no-connect marks 9 -> 11
Other:
- note added: "3.5mm MIDI outputs following the\nTRS MIDI Type A pinning"
Changed lines of the file:
@@
 AR Path="/5F69BED5" Ref="U?"  Part="1"
 AR Path="/5F699A2B/5F69BED5" Ref="U2"  Part="1"
-F 0 "U2" H 3900 3067 50  0000 C CNN
+F 0 "U?" H 3900 3067 50  0000 C CNN
 F 1 "6N138SDM" H 3900 2976 50  0000 C CNN
 F 2 "Package_DIP:SMDIP-8_W9.53mm" H 4190 2300 50  0001 C CNN
@@
 AR Path="/5F69BEDC" Ref="R?"  Part="1"
 AR Path="/5F699A2B/5F69BEDC" Ref="R7"  Part="1"
-F 0 "R7" H 3150 2725 50  0000 C CNN
+F 0 "R?" H 3150 2725 50  0000 C CNN
 F 1 "220" H 3150 2634 50  0000 C CNN
 F 2 "SamacSys_Parts:R_0402_JLCPCB" H 3150 2400 50  0001 C CNN
@@
 AR Path="/5F69BEE4" Ref="R?"  Part="1"
 AR Path="/5F699A2B/5F69BEE4" Ref="R9"  Part="1"
-F 0 "R9" V 4904 2438 50  0000 L CNN
+F 0 "R?" V 4904 2438 50  0000 L CNN
 F 1 "220" V 4995 2438 50  0000 L CNN
 F 2 "SamacSys_Parts:R_0402_JLCPCB" H 4950 2250 50  0001 C CNN
@@
 AR Path="/5F69BEEA" Ref="#PWR?"  Part="1"
 AR Path="/5F699A2B/5F69BEEA" Ref="#PWR041"  Part="1"
-F 0 "#PWR041" H 4950 1950 50  0001 C CNN
+F 0 "#PWR?" H 4950 1950 50  0001 C CNN
 F 1 "+3.3V" H 4965 2273 50  0000 C CNN
 F 2 "" H 4950 2100 50  0001 C CNN
@@
 AR Path="/5F69BEFD" Ref="R?"  Part="1"
 AR Path="/5F699A2B/5F69BEFD" Ref="R8"  Part="1"
-F 0 "R8" V 4604 2838 50  0000 L CNN
+F 0 "R?" V 4604 2838 50  0000 L CNN
 F 1 "10k" V 4695 2838 50  0000 L CNN
 F 2 "SamacSys_Parts:R_0402_JLCPCB" H 5050 2800 50  0001 L CNN
@@
 AR Path="/5F69BF03" Ref="#PWR?"  Part="1"
 AR Path="/5F699A2B/5F69BF03" Ref="#PWR040"  Part="1"
-F 0 "#PWR040" H 4500 2900 50  0001 C CNN
+F 0 "#PWR?" H 4500 2900 50  0001 C CNN
 F 1 "GND" H 4505 2977 50  0000 C CNN
 F 2 "" H 4500 3150 50  0001 C CNN
@@
 AR Path="/5F69BF19" Ref="D?"  Part="1"
 AR Path="/5F699A2B/5F69BF19" Ref="D1"  Part="1"
-F 0 "D1" V 3500 2250 50  0000 L CNN
+F 0 "D?" V 3500 2250 50  0000 L CNN
 F 1 "SM4007PL" V 3600 2150 33  0000 L CNN
 F 2 "SamacSys_Parts:SODFL3718X125N" H 4200 2500 50  0001 L CNN
@@
 U 1 1 5F69C5D0
 P 2600 2400
-F 0 "J13" H 3100 2665 50  0000 C CNN
+F 0 "J?" H 3100 2665 50  0000 C CNN
 F 1 "57PC5F" H 3100 2574 50  0000 C CNN
 F 2 "SamacSys_Parts:57PC5F" H 3450 2500 50  0001 L CNN
@@
 AR Path="/5F69DF4B" Ref="#PWR?"  Part="1"
 AR Path="/5F699A2B/5F69DF4B" Ref="#PWR039"  Part="1"
-F 0 "#PWR039" H 1450 2450 50  0001 C CNN
+F 0 "#PWR?" H 1450 2450 50  0001 C CNN
 F 1 "GND" H 1455 2527 50  0000 C CNN
 F 2 "" H 1450 2700 50  0001 C CNN
@@
 U 1 1 5F6AED33
 P 7900 2400
-F 0 "J14" H 8400 2665 50  0000 C CNN
+F 0 "J?" H 8400 2665 50  0000 C CNN
 F 1 "57PC5F" H 8400 2574 50  0000 C CNN
 F 2 "SamacSys_Parts:57PC5F" H 8750 2500 50  0001 L CNN
@@
 AR Path="/5F6AED3D" Ref="#PWR?"  Part="1"
 AR Path="/5F699A2B/5F6AED3D" Ref="#PWR042"  Part="1"
-F 0 "#PWR042" H 6750 2450 50  0001 C CNN
+F 0 "#PWR?" H 6750 2450 50  0001 C CNN
 F 1 "GND" H 6755 2527 50  0000 C CNN
 F 2 "" H 6750 2700 50  0001 C CNN
@@
 Wire Wire Line
 	6750 2500 6750 2400
-NoConn ~ 7900 2400
 NoConn ~ 7900 2600
 NoConn ~ 6900 2600
@@
 AR Path="/5F6AF8BB" Ref="#PWR?"  Part="1"
 AR Path="/5F699A2B/5F6AF8BB" Ref="#PWR043"  Part="1"
-F 0 "#PWR043" H 8100 2250 50  0001 C CNN
+F 0 "#PWR?" H 8100 2250 50  0001 C CNN
 F 1 "GND" H 8150 2350 50  0000 C CNN
 F 2 "" H 8100 2500 50  0001 C CNN
@@
 AR Path="/5FE8AA11" Ref="#PWR?"  Part="1"
 AR Path="/5F699A2B/5FE8AA11" Ref="#PWR0101"  Part="1"
-F 0 "#PWR0101" H 8950 2550 50  0001 C CNN
+F 0 "#PWR?" H 8950 2550 50  0001 C CNN
 F 1 "+3.3V" H 8965 2873 50  0000 C CNN
 F 2 "" H 8950 2700 50  0001 C CNN
@@
 U 1 1 5FE8D1EA
 P 8350 2700
-F 0 "R10" H 8500 2907 50  0000 C CNN
+F 0 "R?" H 8500 2907 50  0000 C CNN
 F 1 "33" H 8500 2816 50  0000 C CNN
 F 2 "SamacSys_Parts:R_0805_JLCPCB" H 8900 2750 50  0001 L CNN
@@
 U 1 1 5FE8D9B0
 P 8350 3050
-F 0 "R11" H 8500 3257 50  0000 C CNN
+F 0 "R?" H 8500 3257 50  0000 C CNN
 F 1 "10" H 8500 3166 50  0000 C CNN
 F 2 "SamacSys_Parts:R_1206_JLCPCB" H 8900 3100 50  0001 L CNN
@@
 	1    0    0    -1
 $EndComp
+$Comp
+L SamacSys_Parts:SJ1-3523N J?
+U 1 1 5FF42A0E
+P 6950 4000
+F 0 "J?" H 7650 4265 50  0000 C CNN
+F 1 "SJ1-3523N" H 7650 4174 50  0000 C CNN
+F 2 "SJ13523N" H 8200 4100 50  0001 L CNN
+F 3 "https://componentsearchengine.com/Datasheets/1/SJ1-3523N.pdf" H 8200 4000 50  0001 L CNN
+F 4 "Phone Connectors 3.5 MM AUDIO JACK" H 8200 3900 50  0001 L CNN "Description"
+F 5 "5.5" H 8200 3800 50  0001 L CNN "Height"
+F 6 "490-SJ1-3523N" H 8200 3700 50  0001 L CNN "Mouser Part Number"
+F 7 "https://www.mouser.co.uk/ProductDetail/CUI-Devices/SJ1-3523N?qs=WyjlAZoYn50aNl0vAhb3Tg%3D%3D" H 8200 3600 50  0001 L CNN "Mouser Price/Stock"
+F 8 "CUI Devices" H 8200 3500 50  0001 L CNN "Manufacturer_Name"
+F 9 "SJ1-3523N" H 8200 3400 50  0001 L CNN "Manufacturer_Part_Number"
+	1    6950 4000
+	1    0    0    -1
+$EndComp
+$Comp
+L power:GND #PWR?
+U 1 1 5FF42F1C
+P 6800 4000
+AR Path="/5FF42F1C" Ref="#PWR?"  Part="1"
+AR Path="/5F699A2B/5FF42F1C" Ref="#PWR?"  Part="1"
+F 0 "#PWR?" H 6800 3750 50  0001 C CNN
+F 1 "GND" H 6850 3850 50  0000 C CNN
+F 2 "" H 6800 4000 50  0001 C CNN
+F 3 "" H 6800 4000 50  0001 C CNN
+	1    6800 4000
+	1    0    0    -1
+$EndComp
+Wire Wire Line
+	6800 4000 6950 4000
+NoConn ~ 8350 4100
+NoConn ~ 7900 2400
+NoConn ~ 8350 4200
+Text HLabel 8850 4300 2    50   Input ~ 0
+MIDI_OUT2
+$Comp
+L JLCPBC_Basic:10 R?
+U 1 1 5FF49975
+P 8450 4300
+F 0 "R?" H 8600 4507 50  0000 C CNN
+F 1 "10" H 8600 4416 50  0000 C CNN
+F 2 "SamacSys_Parts:R_1206_JLCPCB" H 9000 4350 50  0001 L CNN
+F 3 "https://datasheet.lcsc.com/szlcsc/Uniroyal-Elec-1206W4F100JT5E_C17903.pdf" H 9000 4250 50  0001 L CNN
+F 4 "Chip Resistor - Surface Mount 10Ohms ±1% 1/4W 1206 RoHS" H 9000 4150 50  0001 L CNN "Description"
+F 5 "UNI-ROYAL(Uniroyal Elec)" H 9000 3750 50  0001 L CNN "Manufacturer_Name"
+F 6 "1206W4F100JT5E" H 9000 3650 50  0001 L CNN "Manufacturer_Part_Number"
+F 7 "C17903" H 8450 4300 50  0001 C CNN "JLCPCB Part Number"
+	1    8450 4300
+	1    0    0    -1
+$EndComp
+Wire Wire Line
+	8750 4000 8850 4000
+$Comp
+L power:+3.3V #PWR?
+U 1 1 5FF4B59D
+P 8850 4000
+AR Path="/5FF4B59D" Ref="#PWR?"  Part="1"
+AR Path="/5F699A2B/5FF4B59D" Ref="#PWR?"  Part="1"
+F 0 "#PWR?" H 8850 3850 50  0001 C CNN
+F 1 "+3.3V" H 8865 4173 50  0000 C CNN
+F 2 "" H 8850 4000 50  0001 C CNN
+F 3 "" H 8850 4000 50  0001 C CNN
+	1    8850 4000
+	1    0    0    -1
+$EndComp
+$Comp
+L JLCPBC_Basic:33 R?
+U 1 1 5FF4B5A7
+P 8450 4000
+F 0 "R?" H 8600 4207 50  0000 C CNN
+F 1 "33" H 8600 4116 50  0000 C CNN
+F 2 "SamacSys_Parts:R_0805_JLCPCB" H 9000 4050 50  0001 L CNN
+F 3 "https://datasheet.lcsc.com/szlcsc/Uniroyal-Elec-0805W8F330JT5E_C17634.pdf" H 9000 3950 50  0001 L CNN
+F 4 "Chip Resistor - Surface Mount 33Ohms ±1% 1/8W 0805 RoHS" H 9000 3850 50  0001 L CNN "Description"
+F 5 "UNI-ROYAL(Uniroyal Elec)" H 9000 3450 50  0001 L CNN "Manufacturer_Name"
+F 6 "0805W8F330JT5E" H 9000 3350 50  0001 L CNN "Manufacturer_Part_Number"
+F 7 "C17634" H 8450 4000 50  0001 C CNN "JLCPCB Part Number"
+	1    8450 4000
+	1    0    0    -1
+$EndComp
+Wire Wire Line
+	8350 4000 8450 4000
+Wire Wire Line
+	8350 4300 8450 4300
+Wire Wire Line
+	8750 4300 8850 4300
+Text Notes 7250 3600 0    50   ~ 0
+3.5mm MIDI outputs following the\nTRS MIDI Type A pinning
 $EndSCHEMATC

Commit message: Aligned outputs, started on tracing and connected Pi Innovo header in schematic.
Parts:
- J16: renamed from J?; footprint SJ13523N -> SamacSys_Parts:SJ13523N
- gave numbers to parts that had none: 2
Changed lines of the file:
@@
 $Descr A4 11693 8268
 encoding utf-8
-Sheet 3 4
+Sheet 2 4
 Title ""
 Date ""
@@
 AR Path="/5F69BED5" Ref="U?"  Part="1"
 AR Path="/5F699A2B/5F69BED5" Ref="U2"  Part="1"
-F 0 "U?" H 3900 3067 50  0000 C CNN
+F 0 "U2" H 3900 3067 50  0000 C CNN
 F 1 "6N138SDM" H 3900 2976 50  0000 C CNN
 F 2 "Package_DIP:SMDIP-8_W9.53mm" H 4190 2300 50  0001 C CNN
@@
 AR Path="/5F69BEDC" Ref="R?"  Part="1"
 AR Path="/5F699A2B/5F69BEDC" Ref="R7"  Part="1"
-F 0 "R?" H 3150 2725 50  0000 C CNN
+F 0 "R7" H 3150 2725 50  0000 C CNN
 F 1 "220" H 3150 2634 50  0000 C CNN
 F 2 "SamacSys_Parts:R_0402_JLCPCB" H 3150 2400 50  0001 C CNN
@@
 AR Path="/5F69BEE4" Ref="R?"  Part="1"
 AR Path="/5F699A2B/5F69BEE4" Ref="R9"  Part="1"
-F 0 "R?" V 4904 2438 50  0000 L CNN
+F 0 "R9" V 4904 2438 50  0000 L CNN
 F 1 "220" V 4995 2438 50  0000 L CNN
 F 2 "SamacSys_Parts:R_0402_JLCPCB" H 4950 2250 50  0001 C CNN
@@
 AR Path="/5F69BEEA" Ref="#PWR?"  Part="1"
 AR Path="/5F699A2B/5F69BEEA" Ref="#PWR041"  Part="1"
-F 0 "#PWR?" H 4950 1950 50  0001 C CNN
+F 0 "#PWR041" H 4950 1950 50  0001 C CNN
 F 1 "+3.3V" H 4965 2273 50  0000 C CNN
 F 2 "" H 4950 2100 50  0001 C CNN
@@
 AR Path="/5F69BEFD" Ref="R?"  Part="1"
 AR Path="/5F699A2B/5F69BEFD" Ref="R8"  Part="1"
-F 0 "R?" V 4604 2838 50  0000 L CNN
+F 0 "R8" V 4604 2838 50  0000 L CNN
 F 1 "10k" V 4695 2838 50  0000 L CNN
 F 2 "SamacSys_Parts:R_0402_JLCPCB" H 5050 2800 50  0001 L CNN
@@
 AR Path="/5F69BF03" Ref="#PWR?"  Part="1"
 AR Path="/5F699A2B/5F69BF03" Ref="#PWR040"  Part="1"
-F 0 "#PWR?" H 4500 2900 50  0001 C CNN
+F 0 "#PWR040" H 4500 2900 50  0001 C CNN
 F 1 "GND" H 4505 2977 50  0000 C CNN
 F 2 "" H 4500 3150 50  0001 C CNN
@@
 AR Path="/5F69BF19" Ref="D?"  Part="1"
 AR Path="/5F699A2B/5F69BF19" Ref="D1"  Part="1"
-F 0 "D?" V 3500 2250 50  0000 L CNN
+F 0 "D1" V 3500 2250 50  0000 L CNN
 F 1 "SM4007PL" V 3600 2150 33  0000 L CNN
 F 2 "SamacSys_Parts:SODFL3718X125N" H 4200 2500 50  0001 L CNN
@@
 U 1 1 5F69C5D0
 P 2600 2400
-F 0 "J?" H 3100 2665 50  0000 C CNN
+F 0 "J13" H 3100 2665 50  0000 C CNN
 F 1 "57PC5F" H 3100 2574 50  0000 C CNN
 F 2 "SamacSys_Parts:57PC5F" H 3450 2500 50  0001 L CNN
@@
 AR Path="/5F69DF4B" Ref="#PWR?"  Part="1"
 AR Path="/5F699A2B/5F69DF4B" Ref="#PWR039"  Part="1"
-F 0 "#PWR?" H 1450 2450 50  0001 C CNN
+F 0 "#PWR039" H 1450 2450 50  0001 C CNN
 F 1 "GND" H 1455 2527 50  0000 C CNN
 F 2 "" H 1450 2700 50  0001 C CNN
@@
 U 1 1 5F6AED33
 P 7900 2400
-F 0 "J?" H 8400 2665 50  0000 C CNN
+F 0 "J14" H 8400 2665 50  0000 C CNN
 F 1 "57PC5F" H 8400 2574 50  0000 C CNN
 F 2 "SamacSys_Parts:57PC5F" H 8750 2500 50  0001 L CNN
@@
 AR Path="/5F6AED3D" Ref="#PWR?"  Part="1"
 AR Path="/5F699A2B/5F6AED3D" Ref="#PWR042"  Part="1"
-F 0 "#PWR?" H 6750 2450 50  0001 C CNN
+F 0 "#PWR042" H 6750 2450 50  0001 C CNN
 F 1 "GND" H 6755 2527 50  0000 C CNN
 F 2 "" H 6750 2700 50  0001 C CNN
@@
 AR Path="/5F6AF8BB" Ref="#PWR?"  Part="1"
 AR Path="/5F699A2B/5F6AF8BB" Ref="#PWR043"  Part="1"
-F 0 "#PWR?" H 8100 2250 50  0001 C CNN
+F 0 "#PWR043" H 8100 2250 50  0001 C CNN
 F 1 "GND" H 8150 2350 50  0000 C CNN
 F 2 "" H 8100 2500 50  0001 C CNN
@@
 AR Path="/5FE8AA11" Ref="#PWR?"  Part="1"
 AR Path="/5F699A2B/5FE8AA11" Ref="#PWR0101"  Part="1"
-F 0 "#PWR?" H 8950 2550 50  0001 C CNN
+F 0 "#PWR0101" H 8950 2550 50  0001 C CNN
 F 1 "+3.3V" H 8965 2873 50  0000 C CNN
 F 2 "" H 8950 2700 50  0001 C CNN
@@
 U 1 1 5FE8D1EA
 P 8350 2700
-F 0 "R?" H 8500 2907 50  0000 C CNN
+F 0 "R10" H 8500 2907 50  0000 C CNN
 F 1 "33" H 8500 2816 50  0000 C CNN
 F 2 "SamacSys_Parts:R_0805_JLCPCB" H 8900 2750 50  0001 L CNN
@@
 U 1 1 5FE8D9B0
 P 8350 3050
-F 0 "R?" H 8500 3257 50  0000 C CNN
+F 0 "R11" H 8500 3257 50  0000 C CNN
 F 1 "10" H 8500 3166 50  0000 C CNN
 F 2 "SamacSys_Parts:R_1206_JLCPCB" H 8900 3100 50  0001 L CNN
@@
 $EndComp
 $Comp
-L SamacSys_Parts:SJ1-3523N J?
+L SamacSys_Parts:SJ1-3523N J16
 U 1 1 5FF42A0E
 P 6950 4000
-F 0 "J?" H 7650 4265 50  0000 C CNN
+F 0 "J16" H 7650 4265 50  0000 C CNN
 F 1 "SJ1-3523N" H 7650 4174 50  0000 C CNN
-F 2 "SJ13523N" H 8200 4100 50  0001 L CNN
+F 2 "SamacSys_Parts:SJ13523N" H 8200 4100 50  0001 L CNN
 F 3 "https://componentsearchengine.com/Datasheets/1/SJ1-3523N.pdf" H 8200 4000 50  0001 L CNN
 F 4 "Phone Connectors 3.5 MM AUDIO JACK" H 8200 3900 50  0001 L CNN "Description"
@@
 P 6800 4000
 AR Path="/5FF42F1C" Ref="#PWR?"  Part="1"
-AR Path="/5F699A2B/5FF42F1C" Ref="#PWR?"  Part="1"
-F 0 "#PWR?" H 6800 3750 50  0001 C CNN
+AR Path="/5F699A2B/5FF42F1C" Ref="#PWR0102"  Part="1"
+F 0 "#PWR0102" H 6800 3750 50  0001 C CNN
 F 1 "GND" H 6850 3850 50  0000 C CNN
 F 2 "" H 6800 4000 50  0001 C CNN
@@
 MIDI_OUT2
 $Comp
-L JLCPBC_Basic:10 R?
+L JLCPBC_Basic:10 R16
 U 1 1 5FF49975
 P 8450 4300
-F 0 "R?" H 8600 4507 50  0000 C CNN
+F 0 "R16" H 8600 4500 50  0000 C CNN
 F 1 "10" H 8600 4416 50  0000 C CNN
 F 2 "SamacSys_Parts:R_1206_JLCPCB" H 9000 4350 50  0001 L CNN
@@
 P 8850 4000
 AR Path="/5FF4B59D" Ref="#PWR?"  Part="1"
-AR Path="/5F699A2B/5FF4B59D" Ref="#PWR?"  Part="1"
-F 0 "#PWR?" H 8850 3850 50  0001 C CNN
+AR Path="/5F699A2B/5FF4B59D" Ref="#PWR0103"  Part="1"
+F 0 "#PWR0103" H 8850 3850 50  0001 C CNN
 F 1 "+3.3V" H 8865 4173 50  0000 C CNN
 F 2 "" H 8850 4000 50  0001 C CNN
@@
 $EndComp
 $Comp
-L JLCPBC_Basic:33 R?
+L JLCPBC_Basic:33 R6
 U 1 1 5FF4B5A7
 P 8450 4000
-F 0 "R?" H 8600 4207 50  0000 C CNN
+F 0 "R6" H 8600 4207 50  0000 C CNN
 F 1 "33" H 8600 4116 50  0000 C CNN
 F 2 "SamacSys_Parts:R_0805_JLCPCB" H 9000 4050 50  0001 L CNN
@@
 Wire Wire Line
 	8350 4300 8450 4300
-Wire Wire Line
-	8750 4300 8850 4300
 Text Notes 7250 3600 0    50   ~ 0
 3.5mm MIDI outputs following the\nTRS MIDI Type A pinning
+Wire Wire Line
+	8750 4300 8850 4300
 $EndSCHEMATC
