File: AudioBoard.sch (KiCad schematic (older format))
At the start: 10 parts, among them IC1 AMS1117-5.0, J1 I2S2_OPT, J2 SPI_OPT, J3 Other Teensy pins, J4 UART_OPT, J5 163-179PH-EX, U1 Teensy4.0

Commit message: Updated barreljack (power) footprint and added V_USB selection through jumper.
Parts:
- removed JP1: POWER_SWITCH, Connector_PinSocket_2.54mm:PinSocket_1x02_P2.54mm_Vertical, symbol Device:Jumper_NC_Small
- added JP1: Jumper_NC_Dual, Connector_PinSocket_2.54mm:PinSocket_1x03_P2.54mm_Vertical, symbol Device:Jumper_NC_Dual
- J5: footprint SamacSys_Parts:163179PHEX -> Connector_BarrelJack:BarrelJack_Horizontal
Connections:
- net labels added: V_USB
- wire segments 64 -> 63
- no-connect marks 5 -> 4
Changed lines of the file:
@@
 Wire Wire Line
 	9250 3100 9300 3100
-Wire Wire Line
-	9300 2900 9250 2900
-Wire Wire Line
-	9250 2900 9250 1750
 Text Label 6400 2300 2    50   ~ 0
 5V_EXT
@@
 Wire Wire Line
 	3100 2500 3850 2500
-Wire Wire Line
-	9150 1750 9250 1750
-$Comp
-L Device:Jumper_NC_Small JP1
-U 1 1 5F6C6AB9
-P 9050 1750
-F 0 "JP1" H 9050 1962 50  0000 C CNN
-F 1 "POWER_SWITCH" H 9050 1871 50  0000 C CNN
-F 2 "Connector_PinSocket_2.54mm:PinSocket_1x02_P2.54mm_Vertical" H 9050 1750 50  0001 C CNN
-F 3 "~" H 9050 1750 50  0001 C CNN
-	1    9050 1750
-	1    0    0    -1
-$EndComp
-Wire Wire Line
-	8950 1750 8650 1750
 $Comp
 L SamacSys_Parts:163-179PH-EX J5
@@
 F 0 "J5" H 7600 2050 50  0000 C CNN
 F 1 "163-179PH-EX" H 7750 1650 50  0000 C CNN
-F 2 "SamacSys_Parts:163179PHEX" H 8200 1950 50  0001 L CNN
+F 2 "Connector_BarrelJack:BarrelJack_Horizontal" H 8200 1950 50  0001 L CNN
 F 3 "https://componentsearchengine.com/Datasheets/1/163-179PH-EX.pdf" H 8200 1850 50  0001 L CNN
 F 4 "DC Power Connectors PCB 2.1MM" H 8200 1750 50  0001 L CNN "Description"
@@
 Wire Wire Line
 	8050 1750 8650 1750
-Connection ~ 8650 1750
 Wire Wire Line
 	4250 4250 4250 4750
@@
 F5 "I2S_BCK" O R 3000 5000 50
 $EndSheet
-NoConn ~ 5050 2000
+Text Label 3350 3100 0    50   ~ 0
+I2S_DOUT
+Text Label 3350 3200 0    50   ~ 0
+I2S_DIN
+$Comp
+L Device:Jumper_NC_Dual JP1
+U 1 1 5FEA0033
+P 9300 1750
+F 0 "JP1" V 9254 1852 50  0000 L CNN
+F 1 "Jumper_NC_Dual" V 9345 1852 50  0000 L CNN
+F 2 "Connector_PinSocket_2.54mm:PinSocket_1x03_P2.54mm_Vertical" H 9300 1750 50  0001 C CNN
+F 3 "~" H 9300 1750 50  0001 C CNN
+	1    9300 1750
+	1    0    0    -1
+$EndComp
 $Comp
 L JLCPBC_Basic:AMS1117-5.0 IC?
@@
 	1    0    0    1
 $EndComp
-Text Label 3350 3100 0    50   ~ 0
-I2S_DOUT
-Text Label 3350 3200 0    50   ~ 0
-I2S_DIN
+Text Label 5050 2000 0    50   ~ 0
+V_USB
+Text Label 9650 1750 0    50   ~ 0
+V_USB
+Wire Wire Line
+	8650 1750 9050 1750
+Connection ~ 8650 1750
+Wire Wire Line
+	9300 1850 9300 2900
+Wire Wire Line
+	9550 1750 9650 1750
 $EndSCHEMATC

Commit message: Updated capacitors to smaller/lower voltage ones.
Parts:
- JP1: value Jumper_NC_Dual -> Teensy supply select
Other:
- note added: "This dual jump allows selecting between V_USB and DC_IN after cutting the\nconnection between VIN and VUSB on the back of the Teensy"
- note removed: "To do:\n- On Teensy: cut line between VIN and VUSB on the back!"
Changed lines of the file:
@@
 L power:GND #PWR?
 U 1 1 5F5D1ECA
-P 8650 2300
+P 8650 2050
 AR Path="/5F2A0E47/5F5D1ECA" Ref="#PWR?"  Part="1"
 AR Path="/5F5D1ECA" Ref="#PWR014"  Part="1"
-F 0 "#PWR014" H 8650 2050 50  0001 C CNN
-F 1 "GND" H 8655 2127 50  0000 C CNN
-F 2 "" H 8650 2300 50  0001 C CNN
-F 3 "" H 8650 2300 50  0001 C CNN
-	1    8650 2300
+F 0 "#PWR014" H 8650 1800 50  0001 C CNN
+F 1 "GND" H 8655 1877 50  0000 C CNN
+F 2 "" H 8650 2050 50  0001 C CNN
+F 3 "" H 8650 2050 50  0001 C CNN
+	1    8650 2050
 	1    0    0    -1
 $EndComp
@@
 L power:GND #PWR?
 U 1 1 5F5D1ED4
-P 8650 3550
+P 8650 3300
 AR Path="/5F2A0E47/5F5D1ED4" Ref="#PWR?"  Part="1"
 AR Path="/5F5D1ED4" Ref="#PWR016"  Part="1"
-F 0 "#PWR016" H 8650 3300 50  0001 C CNN
-F 1 "GND" H 8655 3377 50  0000 C CNN
-F 2 "" H 8650 3550 50  0001 C CNN
-F 3 "" H 8650 3550 50  0001 C CNN
-	1    8650 3550
+F 0 "#PWR016" H 8650 3050 50  0001 C CNN
+F 1 "GND" H 8655 3127 50  0000 C CNN
+F 2 "" H 8650 3300 50  0001 C CNN
+F 3 "" H 8650 3300 50  0001 C CNN
+	1    8650 3300
 	1    0    0    -1
 $EndComp
@@
 	1    0    0    -1
 $EndComp
-Text Notes 5750 1200 0    50   ~ 0
-To do:\n- On Teensy: cut line between VIN and VUSB on the back!
+Text Notes 8050 1350 0    50   ~ 0
+This dual jump allows selecting between V_USB and DC_IN after cutting the\nconnection between VIN and VUSB on the back of the Teensy
 Wire Wire Line
 	8250 1950 8050 1950
@@
 U 1 1 5FEA0033
 P 9300 1750
-F 0 "JP1" V 9254 1852 50  0000 L CNN
-F 1 "Jumper_NC_Dual" V 9345 1852 50  0000 L CNN
+F 0 "JP1" H 9200 2000 50  0000 L CNN
+F 1 "Teensy supply select" H 9000 1900 50  0000 L CNN
 F 2 "Connector_PinSocket_2.54mm:PinSocket_1x03_P2.54mm_Vertical" H 9300 1750 50  0001 C CNN
 F 3 "~" H 9300 1750 50  0001 C CNN

Commit message: Replaced one pot by a 3.5mm MIDI Output jack.
Connections:
- net labels added: MIDI_OUT2
- net labels removed: POT6
Changed lines of the file:
@@
 	2350 3600 3850 3600
 NoConn ~ 6050 3600
-Text Label 6450 2600 2    50   ~ 0
-POT6
 Wire Wire Line
 	6450 2600 6050 2600
 Text Label 6450 2700 2    50   ~ 0
-POT5
+POT4
 Wire Wire Line
 	6450 2700 6050 2700
 Text Label 6450 3000 2    50   ~ 0
-POT4
+POT3
 Text Label 6450 3100 2    50   ~ 0
-POT3
-Text Label 6450 3200 2    50   ~ 0
 POT2
+Text Label 6450 2600 2    50   ~ 0
+POT5
 Text Label 6450 3300 2    50   ~ 0
 POT1
@@
 	1    0    0    -1
 $EndComp
-$Sheet
-S 9350 4300 1400 750
-U 5F605664
-F0 "Sheet5F605663" 50
-F1 "Placeholders for IO.sch" 50
-F2 "POT1" O L 9350 4450 50
-F3 "POT4" O L 9350 4750 50
-F4 "POT2" O L 9350 4550 50
-F5 "POT5" O L 9350 4850 50
-F6 "POT6" O L 9350 4950 50
-F7 "POT3" O L 9350 4650 50
-$EndSheet
 Text Label 8850 4450 0    50   ~ 0
 POT1
@@
 Text Label 8850 4650 0    50   ~ 0
 POT3
-Text Label 8850 4950 0    50   ~ 0
-POT6
 Wire Wire Line
 	8850 4450 9350 4450
@@
 Wire Wire Line
 	8850 4850 9350 4850
-Wire Wire Line
-	8850 4950 9350 4950
 $Comp
 L Connector_Generic:Conn_01x06 J2
@@
 $EndComp
 $Sheet
-S 1150 1000 900  500
+S 1150 1000 900  600
 U 5F699A2B
 F0 "MIDI" 50
 F1 "MIDI.sch" 50
 F2 "MIDI_IN" O R 2050 1150 50
-F3 "MIDI_OUT" I R 2050 1350 50
+F3 "MIDI_OUT" I R 2050 1300 50
 $EndSheet
 Wire Wire Line
@@
 Wire Wire Line
 	2050 1150 3250 1150
-Wire Wire Line
-	3100 2500 3100 1350
-Wire Wire Line
-	2050 1350 3100 1350
 Wire Wire Line
 	3100 2500 3850 2500
@@
 Wire Wire Line
 	9550 1750 9650 1750
+Text HLabel 2050 1450 0    50   Output ~ 0
+MIDI_OUT2
+Wire Wire Line
+	2050 1300 3100 1300
+Wire Wire Line
+	3100 1300 3100 2500
+Text Label 2750 1450 2    50   ~ 0
+MIDI_OUT2
+Wire Wire Line
+	2750 1450 2050 1450
+Text Label 6450 3200 2    50   ~ 0
+MIDI_OUT2
+$Sheet
+S 9350 4300 1050 700
+U 5F605664
+F0 "Sheet5F605663" 50
+F1 "Placeholders for IO.sch" 50
+F2 "POT1" O L 9350 4450 50
+F3 "POT4" O L 9350 4750 50
+F4 "POT2" O L 9350 4550 50
+F5 "POT5" O L 9350 4850 50
+F6 "POT3" O L 9350 4650 50
+$EndSheet
 $EndSCHEMATC

Commit message: Aligned outputs, started on tracing and connected Pi Innovo header in schematic.
Parts:
- added J12: Raspberry_Pi_2_3, Connector_PinHeader_2.54mm:PinHeader_2x20_P2.54mm_Vertical, symbol Connector:Raspberry_Pi_2_3
- J5: footprint Connector_BarrelJack:BarrelJack_Horizontal -> SamacSys_Parts:BarrelJack_Horizontal
Connections:
- wire segments 63 -> 83
Other:
- note added: "Note that on the Raspberry Pi 3B+ only one UART is available.\nWe have for now connected MIDI_OUT2 in case we would\nwant to implement a software UART using a regular\n(arbitrarily selected) GPIO pin for now."
Changed lines of the file:
@@
 Wire Wire Line
 	3350 3200 3850 3200
-Text Label 3550 4550 2    50   ~ 0
+Text Label 3100 4300 2    50   ~ 0
 I2S_DOUT
-Text Label 3550 4700 2    50   ~ 0
+Text Label 3100 4450 2    50   ~ 0
 I2S_DIN
 Text Label 6450 2800 2    50   ~ 0
@@
 Text Label 6450 2900 2    50   ~ 0
 I2S_LRCK
-Text Label 3550 5000 2    50   ~ 0
+Text Label 3100 4750 2    50   ~ 0
 I2S_BCK
-Text Label 3550 4850 2    50   ~ 0
+Text Label 3100 4600 2    50   ~ 0
 I2S_LRCK
 Wire Wire Line
-	3000 4550 3550 4550
-Wire Wire Line
-	3000 4700 3550 4700
-Wire Wire Line
-	3550 4850 3000 4850
-Wire Wire Line
-	3000 5000 3550 5000
+	2550 4300 3100 4300
+Wire Wire Line
+	2550 4450 3100 4450
+Wire Wire Line
+	3100 4600 2550 4600
+Wire Wire Line
+	2550 4750 3100 4750
 Wire Wire Line
 	6050 2800 6450 2800
@@
 	6450 3300 6050 3300
 Wire Wire Line
-	6050 3200 6450 3200
-Wire Wire Line
 	6050 3100 6450 3100
 Wire Wire Line
@@
 F2 "MIDI_IN" O R 2050 1150 50
 F3 "MIDI_OUT" I R 2050 1300 50
+F4 "MIDI_OUT2" I R 2050 1450 50
 $EndSheet
 Wire Wire Line
@@
 F 0 "J5" H 7600 2050 50  0000 C CNN
 F 1 "163-179PH-EX" H 7750 1650 50  0000 C CNN
-F 2 "Connector_BarrelJack:BarrelJack_Horizontal" H 8200 1950 50  0001 L CNN
+F 2 "SamacSys_Parts:BarrelJack_Horizontal" H 8200 1950 50  0001 L CNN
 F 3 "https://componentsearchengine.com/Datasheets/1/163-179PH-EX.pdf" H 8200 1850 50  0001 L CNN
 F 4 "DC Power Connectors PCB 2.1MM" H 8200 1750 50  0001 L CNN "Description"
@@
 	4150 4750 4150 4700
 $Sheet
-S 1500 4450 1500 650
+S 1050 4200 1500 650
 U 5F29F5CC
 F0 "Audio IO (I2S)" 50
 F1 "AudioIO.sch" 50
-F2 "I2S_LRCK" O R 3000 4850 50
-F3 "I2S_DIN" I R 3000 4700 50
-F4 "I2S_DOUT" O R 3000 4550 50
-F5 "I2S_BCK" O R 3000 5000 50
+F2 "I2S_LRCK" O R 2550 4600 50
+F3 "I2S_DIN" I R 2550 4450 50
+F4 "I2S_DOUT" O R 2550 4300 50
+F5 "I2S_BCK" O R 2550 4750 50
 $EndSheet
 Text Label 3350 3100 0    50   ~ 0
@@
 Wire Wire Line
 	9550 1750 9650 1750
-Text HLabel 2050 1450 0    50   Output ~ 0
-MIDI_OUT2
 Wire Wire Line
 	2050 1300 3100 1300
 Wire Wire Line
 	3100 1300 3100 2500
-Text Label 2750 1450 2    50   ~ 0
-MIDI_OUT2
-Wire Wire Line
-	2750 1450 2050 1450
-Text Label 6450 3200 2    50   ~ 0
-MIDI_OUT2
 $Sheet
 S 9350 4300 1050 700
@@
 F6 "POT3" O L 9350 4650 50
 $EndSheet
+$Comp
+L Connector:Raspberry_Pi_2_3 J12
+U 1 1 5FF61AF3
+P 3900 6900
+F 0 "J12" V 3050 5400 50  0000 L CNN
+F 1 "Raspberry_Pi_2_3" V 3150 5400 50  0000 L CNN
+F 2 "Connector_PinHeader_2.54mm:PinHeader_2x20_P2.54mm_Vertical" H 3900 6900 50  0001 C CNN
+F 3 "https://www.raspberrypi.org/documentation/hardware/raspberrypi/schematics/rpi_SCH_3bplus_1p0_reduced.pdf" H 3900 6900 50  0001 C CNN
+	1    3900 6900
+	0    1    1    0
+$EndComp
+Wire Wire Line
+	6050 3200 7050 3200
+Wire Wire Line
+	7050 1450 7050 3200
+Wire Wire Line
+	2050 1450 7050 1450
+Text Label 3900 5650 3    50   ~ 0
+I2S_DOUT
+Text Label 4000 5650 3    50   ~ 0
+I2S_DIN
+$Comp
+L power:+3.3V #PWR?
+U 1 1 6002AAD9
+P 5300 7000
+F 0 "#PWR?" H 5300 6850 50  0001 C CNN
+F 1 "+3.3V" H 5315 7173 50  0000 C CNN
+F 2 "" H 5300 7000 50  0001 C CNN
+F 3 "" H 5300 7000 50  0001 C CNN
+	1    5300 7000
+	1    0    0    -1
+$EndComp
+Wire Wire Line
+	5300 7000 5200 7000
+Wire Wire Line
+	5200 7000 5200 7100
+Connection ~ 5200 7000
+Wire Wire Line
+	5200 6700 5200 6800
+$Comp
+L power:+5V #PWR?
+U 1 1 600319A5
+P 5300 6700
+AR Path="/5F2A0E47/600319A5" Ref="#PWR?"  Part="1"
+AR Path="/600319A5" Ref="#PWR?"  Part="1"
+F 0 "#PWR?" H 5300 6550 50  0001 C CNN
+F 1 "+5V" H 5315 6873 50  0000 C CNN
+F 2 "" H 5300 6700 50  0001 C CNN
+F 3 "" H 5300 6700 50  0001 C CNN
+	1    5300 6700
+	1    0    0    -1
+$EndComp
+Wire Wire Line
+	5200 6700 5300 6700
+Connection ~ 5200 6700
+Text Label 4800 5650 3    50   ~ 0
+MIDI_OUT
+Text Label 3700 5650 3    50   ~ 0
+MIDI_OUT2
+Text Label 4700 5650 3    50   ~ 0
+MIDI_IN
+Text Label 6450 3200 2    50   ~ 0
+MIDI_OUT2
+Text Label 4100 5650 3    50   ~ 0
+I2S_LRCK
+Text Label 4300 5650 3    50   ~ 0
+I2S_BCK
+$Comp
+L power:GND #PWR?
+U 1 1 60033F69
+P 2500 7200
+F 0 "#PWR?" H 2500 6950 50  0001 C CNN
+F 1 "GND" H 2505 7027 50  0000 C CNN
+F 2 "" H 2500 7200 50  0001 C CNN
+F 3 "" H 2500 7200 50  0001 C CNN
+	1    2500 7200
+	1    0    0    -1
+$EndComp
+Wire Wire Line
+	2600 6500 2600 6600
+Connection ~ 2600 6600
+Wire Wire Line
+	2600 6600 2600 6700
+Connection ~ 2600 6700
+Wire Wire Line
+	2600 6700 2600 6800
+Connection ~ 2600 6800
+Wire Wire Line
+	2600 6800 2600 6900
+Connection ~ 2600 6900
+Wire Wire Line
+	2600 6900 2600 7000
+Connection ~ 2600 7000
+Wire Wire Line
+	2600 7000 2600 7100
+Connection ~ 2600 7100
+Wire Wire Line
+	2600 7100 2600 7200
+Wire Wire Line
+	2500 7200 2600 7200
+Connection ~ 2600 7200
+Wire Wire Line
+	4100 5650 4100 6100
+Wire Wire Line
+	4300 5650 4300 6100
+Wire Wire Line
+	3900 5650 3900 6100
+Wire Wire Line
+	4000 5650 4000 6100
+Wire Wire Line
+	4800 5650 4800 6100
+Wire Wire Line
+	4700 5650 4700 6100
+Wire Wire Line
+	3700 5650 3700 6100
+Text Notes 1150 5950 0    50   ~ 0
+Note that on the Raspberry Pi 3B+ only one UART is available.\nWe have for now connected MIDI_OUT2 in case we would\nwant to implement a software UART using a regular\n(arbitrarily selected) GPIO pin for now.
 $EndSCHEMATC

Commit message: Updated PCB traces.
Connections:
- no-connect marks 4 -> 25
Changed lines of the file:
@@
 Text Notes 1150 5950 0    50   ~ 0
 Note that on the Raspberry Pi 3B+ only one UART is available.\nWe have for now connected MIDI_OUT2 in case we would\nwant to implement a software UART using a regular\n(arbitrarily selected) GPIO pin for now.
+NoConn ~ 3200 6100
+NoConn ~ 3300 6100
+NoConn ~ 3400 6100
+NoConn ~ 3500 6100
+NoConn ~ 3600 6100
+NoConn ~ 4400 6100
+NoConn ~ 4500 6100
+NoConn ~ 4800 7700
+NoConn ~ 4700 7700
+NoConn ~ 4500 7700
+NoConn ~ 4400 7700
+NoConn ~ 4200 7700
+NoConn ~ 4100 7700
+NoConn ~ 4000 7700
+NoConn ~ 3800 7700
+NoConn ~ 3700 7700
+NoConn ~ 3600 7700
+NoConn ~ 3500 7700
+NoConn ~ 3400 7700
+NoConn ~ 3200 7700
+NoConn ~ 3100 7700
 $EndSCHEMATC
