File: AudioIO.sch (KiCad schematic (older format))
At the start: 34 parts, among them IC2 PCM5102APWR, IC3 PCM1803ADBR, J15 RCA_2x2, U3 24.576MHz

Commit message: Updated I2S crystal/oscillator
Parts:
- removed C31: 10nF50V, SamacSys_Parts:CAPC2012X65N, symbol JLCPBC_Basic:10nF50V
- removed U3: 24.576MHz, Crystal:Crystal_SMD_3225-4Pin_3.2x2.5mm, symbol JLCPCB_Extended:24.576MHz
- added C?: 10uF25V, CAPC2012X145N, symbol JLCPBC_Basic:10uF25V
- added JP?: OSC_DIS, Connector_PinSocket_2.54mm:PinSocket_1x02_P2.54mm_Vertical, symbol Device:Jumper_NC_Small
- added R?: 10k, SamacSys_Parts:R_0402_JLCPCB, symbol JLCPBC_Basic:10k
- added TP?: TestPoint, symbol Connector:TestPoint
- added U?: 24.576MHz, Crystal:Crystal_SMD_3225-4Pin_3.2x2.5mm, symbol JLCPCB_Extended:24.576MHz
Connections:
- wire segments 104 -> 107
Changed lines of the file:
@@
 	6000 1650 5800 1650
-$Comp
-L JLCPCB_Extended:24.576MHz U3
-U 1 1 5F3971E3
-P 9800 1400
-F 0 "U3" H 9800 1675 50  0000 C CNN
-F 1 "24.576MHz" H 9800 1584 50  0000 C CNN
-F 2 "Crystal:Crystal_SMD_3225-4Pin_3.2x2.5mm" H 9800 1150 50  0001 C CNN
-F 3 "https://datasheet.lcsc.com/szlcsc/Yangxing-Tech-O322524576MEEA4SC_C27869.pdf" H 9800 1400 50  0001 C CNN
-F 4 "C27869" H 9800 1050 50  0001 C CNN "JLCPCB Part Number"
-	1    9800 1400
-	-1   0    0    -1
-$EndComp
-Wire Wire Line
-	10100 1450 10100 1350
-$Comp
-L JLCPBC_Basic:10nF50V C31
-U 1 1 5F3B2686
-P 9550 1850
-F 0 "C31" H 9800 2115 50  0000 C CNN
-F 1 "10nF50V" H 9800 2024 50  0000 C CNN
-F 2 "SamacSys_Parts:CAPC2012X65N" H 9900 1900 50  0001 L CNN
-F 3 "" H 9900 1800 50  0001 L CNN
-F 4 "Samsung Electro-Mechanics 0805 CL 10nF Ceramic Multilayer Capacitor, 50 V, +125C, X7R Dielectric, +/-10% SMD" H 9900 1700 50  0001 L CNN "Description"
-F 5 "0.65" H 9900 1600 50  0001 L CNN "Height"
-F 6 "N/A" H 9900 1500 50  0001 L CNN "Mouser Part Number"
-F 7 "https://www.mouser.co.uk/ProductDetail/Samsung-Electro-Mechanics/CL21B103KBANNNC?qs=349EhDEZ59oTK9iJ%2FqCMuw%3D%3D" H 9900 1400 50  0001 L CNN "Mouser Price/Stock"
-F 8 "Samsung Electro-Mechanics" H 9900 1300 50  0001 L CNN "Manufacturer_Name"
-F 9 "CL21B103KBANNNC" H 9900 1200 50  0001 L CNN "Manufacturer_Part_Number"
-F 10 "C1710" H 9550 1850 50  0001 C CNN "JLCPCB Part Number"
-	1    9550 1850
-	1    0    0    -1
-$EndComp
-Wire Wire Line
-	10050 1850 10100 1850
-Wire Wire Line
-	10100 1850 10100 1450
-Connection ~ 10100 1450
-Wire Wire Line
-	9500 1450 9500 1850
-Wire Wire Line
-	9500 1850 9550 1850
-$Comp
-L power:GND #PWR069
-U 1 1 5F3C4DE7
-P 9500 1850
-F 0 "#PWR069" H 9500 1600 50  0001 C CNN
-F 1 "GND" H 9505 1677 50  0000 C CNN
-F 2 "" H 9500 1850 50  0001 C CNN
-F 3 "" H 9500 1850 50  0001 C CNN
-	1    9500 1850
-	1    0    0    -1
-$EndComp
-Connection ~ 9500 1850
 $Comp
 L power:GND #PWR048
@@
 Text Notes 4200 950  0    50   ~ 0
 I2S ADC
-Text Label 9300 1350 0    50   ~ 0
+Text Label 7450 2050 2    50   ~ 0
 SCK
 Wire Wire Line
-	9300 1350 9500 1350
-Text Label 7650 2050 2    50   ~ 0
-SCK
-Wire Wire Line
-	7200 2050 7650 2050
+	7200 2050 7550 2050
 $Comp
 L power:+3.3V #PWR059
@@
 Wire Wire Line
 	8000 4500 9100 4500
+$Comp
+L JLCPCB_Extended:24.576MHz U?
+U 1 1 5FE94DFB
+P 9900 1500
+F 0 "U?" H 9900 1775 50  0000 C CNN
+F 1 "24.576MHz" H 9900 1684 50  0000 C CNN
+F 2 "Crystal:Crystal_SMD_3225-4Pin_3.2x2.5mm" H 9900 1250 50  0001 C CNN
+F 3 "https://datasheet.lcsc.com/szlcsc/Yangxing-Tech-O322524576MEEA4SC_C27869.pdf" H 9900 1500 50  0001 C CNN
+F 4 "C27869" H 9900 1150 50  0001 C CNN "JLCPCB Part Number"
+	1    9900 1500
+	1    0    0    -1
+$EndComp
+$Comp
+L Device:Jumper_NC_Small JP?
+U 1 1 5FE91BBF
+P 9400 1550
+F 0 "JP?" H 9400 1400 50  0000 C CNN
+F 1 "OSC_DIS" H 9400 1500 50  0000 C CNN
+F 2 "Connector_PinSocket_2.54mm:PinSocket_1x02_P2.54mm_Vertical" H 9400 1550 50  0001 C CNN
+F 3 "~" H 9400 1550 50  0001 C CNN
+	1    9400 1550
+	1    0    0    1
+$EndComp
+$Comp
+L power:GND #PWR069
+U 1 1 5F3C4DE7
+P 9600 1850
+F 0 "#PWR069" H 9600 1600 50  0001 C CNN
+F 1 "GND" H 9605 1677 50  0000 C CNN
+F 2 "" H 9600 1850 50  0001 C CNN
+F 3 "" H 9600 1850 50  0001 C CNN
+	1    9600 1850
+	1    0    0    -1
+$EndComp
+Wire Wire Line
+	10200 1450 10400 1450
+Text Label 10400 1450 2    50   ~ 0
+SCK
+$Comp
+L power:+3.3V #PWR?
+U 1 1 5FEA6972
+P 9200 1300
+F 0 "#PWR?" H 9200 1150 50  0001 C CNN
+F 1 "+3.3V" H 9215 1473 50  0000 C CNN
+F 2 "" H 9200 1300 50  0001 C CNN
+F 3 "" H 9200 1300 50  0001 C CNN
+	1    9200 1300
+	1    0    0    -1
+$EndComp
+$Comp
+L JLCPBC_Basic:10uF25V C?
+U 1 1 5FEAFA4D
+P 9200 1550
+F 0 "C?" V 9300 1300 50  0000 L CNN
+F 1 "10uF25V" V 9400 1100 50  0000 L CNN
+F 2 "CAPC2012X145N" H 9450 1600 50  0001 L CNN
+F 3 "http://www.farnell.com/datasheets/2710652.pdf?_ga=2.232319711.1701824318.1596544434-371254432.1596544434" H 9450 1500 50  0001 L CNN
+F 4 "Samsung" H 9450 1400 50  0001 L CNN "Description"
+F 5 "1.45" H 9450 1300 50  0001 L CNN "Height"
+F 6 "N/A" H 9450 1200 50  0001 L CNN "Mouser Part Number"
+F 7 "https://www.mouser.co.uk/ProductDetail/Samsung-Electro-Mechanics/CL21A106KAYNNNE?qs=yOVawPpwOwmTXAd4dJtNjA%3D%3D" H 9450 1100 50  0001 L CNN "Mouser Price/Stock"
+F 8 "Samsung Electro-Mechanics" H 9450 1000 50  0001 L CNN "Manufacturer_Name"
+F 9 "CL21A106KAYNNNE" H 9450 900 50  0001 L CNN "Manufacturer_Part_Number"
+F 10 "C15850" H 9200 1400 50  0001 C CNN "JLCPCB Part Number"
+	1    9200 1550
+	0    1    1    0
+$EndComp
+$Comp
+L JLCPBC_Basic:10k R?
+U 1 1 5FEC6DE4
+P 9600 1550
+F 0 "R?" V 9704 1620 50  0000 L CNN
+F 1 "10k" V 9795 1620 50  0000 L CNN
+F 2 "SamacSys_Parts:R_0402_JLCPCB" H 10150 1600 50  0001 L CNN
+F 3 "https://datasheet.lcsc.com/szlcsc/Uniroyal-Elec-0402WGF1002TCE_C25744.pdf" H 10150 1500 50  0001 L CNN
+F 4 "Chip Resistor - Surface Mount 10KOhms +/-1% 1/16W 0402 RoHS" H 10150 1400 50  0001 L CNN "Description"
+F 5 "0.4" H 10150 1300 50  0001 L CNN "Height"
+F 6 "UNI-ROYAL(Uniroyal Elec)" H 10150 1000 50  0001 L CNN "Manufacturer_Name"
+F 7 "0402WGF1002TCE" H 10150 900 50  0001 L CNN "Manufacturer_Part_Number"
+F 8 "C25744" H 9600 1550 50  0001 C CNN "JLCPCB Part Number"
+	1    9600 1550
+	0    1    1    0
+$EndComp
+Wire Wire Line
+	9500 1550 9600 1550
+Connection ~ 9600 1550
+Wire Wire Line
+	9300 1550 9200 1550
+Wire Wire Line
+	9200 1550 9200 1300
+Connection ~ 9200 1550
+Connection ~ 9600 1850
+Wire Wire Line
+	9200 1850 9600 1850
+Wire Wire Line
+	10200 1550 10200 1850
+Wire Wire Line
+	9600 1850 10200 1850
+Wire Wire Line
+	9600 1450 9600 1300
+Wire Wire Line
+	9600 1300 9200 1300
+Connection ~ 9200 1300
+$Comp
+L Connector:TestPoint TP?
+U 1 1 5FEF80D5
+P 7550 2050
+F 0 "TP?" H 7608 2168 50  0000 L CNN
+F 1 "TestPoint" H 7608 2077 50  0000 L CNN
+F 2 "" H 7750 2050 50  0001 C CNN
+F 3 "~" H 7750 2050 50  0001 C CNN
+	1    7550 2050
+	1    0    0    -1
+$EndComp
 $EndSCHEMATC

Commit message: Updated capacitors to smaller/lower voltage ones.
Parts:
- removed C10, C20, C21, C22, C26, C27, C9: 10uF25V, SamacSys_Parts:CAPC2012X145N, symbol JLCPBC_Basic:10uF25V
- removed C11, C12: 1uF50V, SamacSys_Parts:CAPC2012X135N, symbol JLCPBC_Basic:1uF50V
- removed C13, C14, C17, C18, C24, C25, C30: 100nF50V, SamacSys_Parts:CAPC3216X100N, symbol JLCPBC_Basic:100nF50V
- removed C?: 10uF25V, CAPC2012X145N, symbol JLCPBC_Basic:10uF25V
- added C? (x8): 100nF16V, CAPC1005X55N, symbol JLCPBC_Basic:100nF16V
- added C? (x2): 1uF25V, CAPC1005X60N, symbol JLCPBC_Basic:1uF25V
- added C? (x7): 10uF6.3V, CAPC1005X70N, symbol JLCPBC_Basic:10uF6.3V
Other:
- moved on the sheet: C16

Commit message: Aligned outputs, started on tracing and connected Pi Innovo header in schematic.
Parts:
- C10, C14, C17, C21, C22, C7, C8, C9: renamed from C?; footprint CAPC1005X55N -> SamacSys_Parts:CAPC1005X55N
- C11, C12, C13, C18, C20, C3, C4: renamed from C?; footprint CAPC1005X70N -> SamacSys_Parts:CAPC1005X70N
- C5, C6: renamed from C?; footprint CAPC1005X60N -> SamacSys_Parts:CAPC1005X60N
- TP1: renamed from TP?; footprint (none) -> Connector_PinHeader_2.54mm:PinHeader_1x01_P2.54mm_Vertical
- gave numbers to parts that had none: 3

Commit message: Added pin header for I2S input, to connect an external ADC (the PCM1803ADBR was unavailable at the time of ordering).
Parts:
- added J17: Conn_01x06, Connector_PinHeader_2.54mm:PinHeader_1x06_P2.54mm_Vertical, symbol Connector_Generic:Conn_01x06
Connections:
- wire segments 107 -> 113
Changed lines of the file:
@@
 Text HLabel 1750 5600 0    50   Input ~ 0
 I2S_LRCK
-Text HLabel 7300 2350 2    50   Output ~ 0
+Text HLabel 7500 2350 2    50   Output ~ 0
 I2S_DIN
 Text HLabel 1750 5700 0    50   Input ~ 0
@@
 	2700 6000 2700 5900
 Connection ~ 2700 6000
-Text HLabel 5700 2450 0    50   Input ~ 0
+Text HLabel 5550 2450 0    50   Input ~ 0
 I2S_LRCK
 Wire Wire Line
-	5700 2450 6000 2450
-Wire Wire Line
 	1750 5800 2700 5800
-Text HLabel 7300 2450 2    50   Input ~ 0
+Text HLabel 7500 2450 2    50   Input ~ 0
 I2S_BCK
 $Comp
@@
 Wire Wire Line
 	8000 2450 8000 2500
-Wire Wire Line
-	7200 2350 7300 2350
-Wire Wire Line
-	7200 2450 7300 2450
 $Comp
 L power:+3.3V #PWR066
@@
 $EndComp
 Connection ~ 1400 4850
+$Comp
+L Connector_Generic:Conn_01x06 J17
+U 1 1 5FEBF30D
+P 4400 3400
+F 0 "J17" V 4272 3680 50  0000 L CNN
+F 1 "Conn_01x06" V 4363 3680 50  0000 L CNN
+F 2 "Connector_PinHeader_2.54mm:PinHeader_1x06_P2.54mm_Vertical" H 4400 3400 50  0001 C CNN
+F 3 "~" H 4400 3400 50  0001 C CNN
+	1    4400 3400
+	0    1    1    0
+$EndComp
+$Comp
+L power:+5V #PWR0108
+U 1 1 5FEC11FB
+P 4600 2800
+F 0 "#PWR0108" H 4600 2650 50  0001 C CNN
+F 1 "+5V" H 4615 2973 50  0000 C CNN
+F 2 "" H 4600 2800 50  0001 C CNN
+F 3 "" H 4600 2800 50  0001 C CNN
+	1    4600 2800
+	1    0    0    -1
+$EndComp
+$Comp
+L power:GND #PWR0109
+U 1 1 5FEC158E
+P 4500 2800
+F 0 "#PWR0109" H 4500 2550 50  0001 C CNN
+F 1 "GND" V 4505 2672 50  0000 R CNN
+F 2 "" H 4500 2800 50  0001 C CNN
+F 3 "" H 4500 2800 50  0001 C CNN
+	1    4500 2800
+	-1   0    0    1
+$EndComp
+Text Label 5600 2450 0    50   ~ 0
+I2S_LRCK
+Wire Wire Line
+	5550 2450 6000 2450
+Text Label 4400 2800 3    50   ~ 0
+I2S_LRCK
+Wire Wire Line
+	4400 3200 4400 2800
+Wire Wire Line
+	4600 2800 4600 3200
+Wire Wire Line
+	4500 2800 4500 3200
+Text Label 7200 2350 0    50   ~ 0
+I2S_DIN
+Wire Wire Line
+	7200 2350 7500 2350
+Wire Wire Line
+	7200 2450 7500 2450
+Text Label 7200 2450 0    50   ~ 0
+I2S_BCK
+Text Label 4200 2800 3    50   ~ 0
+I2S_BCK
+Wire Wire Line
+	4200 2800 4200 3200
+Text Label 4300 2800 3    50   ~ 0
+I2S_DIN
+Wire Wire Line
+	4300 2800 4300 3200
+Text Label 4100 2800 3    50   ~ 0
+SCK
+Wire Wire Line
+	4100 2800 4100 3200
 $EndSCHEMATC
